File: Hardware/IOT-Temprature-Sensor.kicad_pcb (KiCad board)
At the start: 4 copper layers, 31 x 23.4 mm, 77 parts, among them IC1 AP7366-33SN-7, IC2 BMA423, IC3 NST1001, J1 Conn_01x04_Male, J3 Conn_01x02, Q1 MMBT3904, Q2 MMBT3904, Q3 CJE3139K, SW1 SW_1003B, SW2 SW_1003B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

Commit message: xiaoming-opensource
Connections:
- R22 pad 2: /GPIO22 -> (no net)
Routing:
- net /GPIO22: track 7.34 -> 0.00 mm, vias 1 -> 0
- net (no net): track 0.00 -> 7.34 mm, vias 0 -> 1

Commit message: xiaoming-opensource
Parts:
- removed C20, C21, C22, C26, C27, C35, C39: 0.1uF, Capacitor_SMD:C_0402_1005Metric
- removed C36, C38: 10uF, Capacitor_SMD:C_0402_1005Metric
- removed C37: 10nF, Capacitor_SMD:C_0402_1005Metric
- removed IC3: NST1001, Sensor_Voltage:NST1001NEW
- removed R13, R14: 1.2K, Resistor_SMD:R_0402_1005Metric
- removed R8: 50K, Resistor_SMD:R_0402_1005Metric
- removed U2: PAH8011-ETLGA, Package_DFN_QFN:PAH8011ET
- removed U5: SGM2031-1.8YUDH4G/TR, Package_DFN_QFN:SMG2033-DFN
- R5: value 800K -> 680K
- R7: value 50K -> 47K
- renumbered Q3 to Q1, Q1 to Q2, Q2 to Q3, Y3 to Y1
Connections:
- R22 pad 2: (no net) -> /GPIO22
- U1 pad 28: /GPIO6 -> (no net)
- U1 pad 31: /GPIO7 -> (no net)
- U1 pad 47: /AS_EN -> (no net)
Routing:
- net /GPIO22: track 0.00 -> 7.34 mm, vias 0 -> 1
- net (no net): track 7.34 -> 0.00 mm, vias 1 -> 0

Commit message: xiaoming-opensource
Parts:
- removed R11: 30K, Resistor_SMD:R_0402_1005Metric
Routing:
- net /GPIO6: track 17.7 -> 0.00 mm, vias 2 -> 0
- net /GPIO7: track 13.2 -> 0.00 mm, vias 2 -> 0
- net +1V8: track 13.1 -> 0.00 mm, vias 1 -> 0
- net +3V3: track 169.0 -> 157.6 mm, vias 12 -> 11
- net /I2C_SDA: track 16.9 -> 5.72 mm
- net /I2C_SCL: track 19.5 -> 8.50 mm
- net /AS_EN: track 8.73 -> 0.00 mm, vias 2 -> 0
- net /GPIO22: track 7.34 -> 5.17 mm
- net /GPIO5_ADC5: track 18.8 -> 16.7 mm
- net Net-(C20-Pad1): track 1.61 -> 0.00 mm, vias 1 -> 0
Other:
- outline, holes or cut-outs redrawn
